Commit message: Imported upstream version '1.23.2' of 'upstream'

File: pal_sea_arm_description/robots/pal_sea_arm.urdf.xacro (robot description, xacro)
@@ -29,4 +29,5 @@
   <xacro:arg name="use_sim_time" default="False"/>
   <xacro:arg name="namespace" default=""/>
+  <xacro:arg name="gazebo_version" default="classic"/>
   <!-- Mujoco args -->
   <xacro:arg name="sim_type" default="gazebo" />
@@ -41,4 +42,5 @@
   <xacro:property name="tool_changer" value="$(arg tool_changer)" />
   <xacro:property name="nsp" value="$(arg namespace)" />
+  <xacro:property name="gazebo_version" value="$(arg gazebo_version)"/>
   <xacro:property name="sim_type" value="$(arg sim_type)" />
   <xacro:property name="mj_control" value="$(arg mj_control)"/>

File: pal_sea_arm_description/urdf/arm/arm_limits/tiago-pro/straight-wrist.limits.xacro (robot description, xacro)
@@ -1,8 +1,8 @@
 <robot xmlns:xacro="http://ros.org/wiki/xacro">
   <!-- Joint limits -->
-  <xacro:property name="arm_5_joint_ub" value="150" />
-  <xacro:property name="arm_5_joint_lb" value="-150" />
-  <xacro:property name="arm_6_joint_ub" value="115" />
-  <xacro:property name="arm_6_joint_lb" value="-115" />
+  <xacro:property name="arm_5_joint_ub" value="${210 if joint_reflect == 1 else 90}" />
+  <xacro:property name="arm_5_joint_lb" value="${-90 if joint_reflect == 1 else -210}" />
+  <xacro:property name="arm_6_joint_ub" value="120" />
+  <xacro:property name="arm_6_joint_lb" value="-120" />
   <xacro:property name="arm_7_joint_ub" value="150" />
   <xacro:property name="arm_7_joint_lb" value="-150" />

File: pal_sea_arm_description/urdf/end_effector/end_effector.urdf.xacro (robot description, xacro)
@@ -20,9 +20,9 @@
     - reflect: Set to 1 for a right end effector, or to -1 for a left end effector
   -->
-  <xacro:macro name="pal_sea_arm_end_effector" params="name parent type tool_changer reflect">
+  <xacro:macro name="pal_sea_arm_end_effector" params="name parent type tool_changer reflect calibration_tool:=False">
     <!-- PAL Pro Gripper -->
     <xacro:if value="${type == 'pal-pro-gripper'}">
       <xacro:include filename="$(find pal_pro_gripper_description)/urdf/gripper.urdf.xacro" />
-      <xacro:pal_pro_gripper name="${name}" parent="${parent}" tool_changer="${tool_changer}">
+      <xacro:pal_pro_gripper name="${name}" parent="${parent}" tool_changer="${tool_changer}" calibration_tool="${calibration_tool}">
         <origin xyz="0.0 0.0 0.0" rpy="0 0 0"/>
       </xacro:pal_pro_gripper>

Commit message: Imported upstream version '2.6.0' of 'upstream'

File: pal_sea_arm_description/robots/pal_sea_arm.urdf.xacro (robot description, xacro)
@@ -34,4 +34,6 @@
   <xacro:arg name="mj_control" default="false" />
   <xacro:arg name="world_name" default="floor" />
+  <!-- Limits v2-->
+  <xacro:arg name="limits_v2" default="False"/>
   <!-- PROPERTIES -->
   <xacro:property name="end_effector" value="$(arg end_effector)" />
@@ -41,6 +43,7 @@
   <xacro:property name="torque_estimation" value="$(arg torque_estimation)" />
   <xacro:property name="tool_changer" value="$(arg tool_changer)" />
-  <xacro:property name="nsp" value="$(arg namespace)" />
+  <xacro:property name="namespace" value="$(arg namespace)" />
   <xacro:property name="gazebo_version" value="$(arg gazebo_version)"/>
+  <xacro:property name="limits_v2" value="$(arg limits_v2)"/>
   <xacro:property name="sim_type" value="$(arg sim_type)" />
   <xacro:property name="mj_control" value="$(arg mj_control)"/>
@@ -49,5 +52,5 @@
     <xacro:wrong_end_effector/>
   </xacro:if>
-  <xacro:if value="${wrist_model not in ['straight-wrist', 'spherical-wrist']}">
+  <xacro:if value="${wrist_model not in ['straight-wrist', 'spherical-wrist', 'short-wrist']}">
     <xacro:wrong_wrist_model/>
   </xacro:if>
@@ -88,28 +91,42 @@
   </xacro:if>
   <!-- ROBOT DEFINITION -->
-  <link name="world"/>
-  <joint name="world_fixed" type="fixed">
-    <origin xyz="0 0 0" rpy="0 0 0"/>
+  <link name="world"></link>
+  <joint name="base_joint" type="fixed">
+    <origin xyz="0 0 0.05" rpy="0 0 0"/>
     <parent link="world"/>
+    <child link="base_link"/>
+  </joint>
+  <link name="base_link">
+    <inertial>
+      <origin xyz="0 0 -0.1" rpy="0 0 0"/>
+      <mass value="0.01" />
+      <inertia ixx="0.001" ixy="0" ixz="0" iyy="0.001" iyz="0" izz="0.001"/>
+    </inertial>
+  </link>
+  <!-- ARM ROOT LINK -->
+  <joint name="arm_root_joint" type="fixed">
+    <origin xyz="0 0 1.272" rpy="0 0 0"/>
+    <parent link="base_link"/>
     <child link="arm_root_link"/>
   </joint>
-  <!-- BASE LINK -->
   <link name="arm_root_link">
     <inertial>
-      <origin xyz="0.0 0.0 0.0" rpy="0 0 0" />
-      <mass value="0.28971" />
-      <inertia ixx="0.00022379" ixy="1.5836E-20" ixz="5.2063E-21" iyy="0.00022379" iyz="-5.1333E-21" izz="0.00019673" />
+      <origin xyz="-0.0023663 -0.0013678 -0.86311" rpy="0 0 2.618" />
+      <mass value="89.317"/>
+      <inertia ixx="6.284" ixy="-2.737E-05" ixz="0.0010106" iyy="6.2841" iyz="0.00058347" izz="3.768" />
     </inertial>
     <visual>
-      <origin xyz="0 0 0" rpy="0 0 0" />
+      <origin xyz="0 0 -0.08" rpy="0 0 2.618 " />
       <geometry>
-        <mesh filename="package://pal_sea_arm_description/meshes/arm_tiago_pro/arm_base_link.stl" />
+        <mesh filename="package://pal_sea_arm_description/meshes/pal_sea_arm_standalone/base_link.stl" />
       </geometry>
-      <material name="pal/DarkGrey"/>
+      <material name="">
+        <color rgba="0.89412 0.91373 0.92941 1" />
+      </material>
     </visual>
     <collision>
-      <origin xyz="0 0 0" rpy="0 0 0" />
+      <origin xyz="0 0 -0.08" rpy="0 0 2.618" />
       <geometry>
-        <mesh filename="package://pal_sea_arm_description/meshes/arm_tiago_pro/arm_base_link.stl" />
+        <mesh filename="package://pal_sea_arm_description/meshes/pal_sea_arm_standalone/base_link.stl" />
       </geometry>
     </collision>
@@ -121,6 +138,6 @@
   </gazebo>
   <!-- ARM -->
-  <xacro:pal_sea_arm name="arm" parent="arm_root_link" arm_type="${arm_type}" tool_changer="${tool_changer}" wrist_model="${wrist_model}" reflect="1" arm_1_offset="0" arm_2_offset="0" arm_3_offset="0" arm_4_offset="0" arm_5_offset="0" arm_6_offset="0" arm_7_offset="0">
-    <origin xyz="0 0 0" rpy="0 0 3.1416" />
+  <xacro:pal_sea_arm name="arm" parent="arm_root_link" arm_type="${arm_type}" tool_changer="${tool_changer}" wrist_model="${wrist_model}" reflect="1" arm_1_offset="0" arm_2_offset="0" arm_3_offset="0" arm_4_offset="0" arm_5_offset="0" arm_6_offset="0" arm_7_offset="0" limits_v2="${limits_v2}">
+    <origin xyz="0.140 0 -0.08" rpy="0 0 0" />
   </xacro:pal_sea_arm>
   <!-- Force Torque sensor-->
@@ -163,4 +180,4 @@
   </xacro:if>
   <!-- ROS2 control -->
-  <xacro:pal_sea_arm_ros2_control use_sim_time="$(arg use_sim_time)" torque_estimation="${torque_estimation}"/>
+  <xacro:pal_sea_arm_ros2_control use_sim_time="$(arg use_sim_time)" torque_estimation="${torque_estimation}" gazebo_version="${gazebo_version}"/>
 </robot>

File: pal_sea_arm_description/ros2_control/ros2_control.urdf.xacro (robot description, xacro)
@@ -13,5 +13,5 @@
  -->
 <robot xmlns:xacro="http://ros.org/wiki/xacro" name="pal_sea_arm">
-  <xacro:macro name="pal_sea_arm_ros2_control" params="use_sim_time:=^|false torque_estimation:=false sim_type:=no-simulation">
+  <xacro:macro name="pal_sea_arm_ros2_control" params="use_sim_time:=^|false torque_estimation:=false sim_type:=gazebo gazebo_version:=classic">
     <xacro:arg name="end_effector" default="no-end-effector"/>
     <xacro:arg name="ft_sensor" default="no-ft-sensor"/>
@@ -33,9 +33,16 @@
           </xacro:if>
           <xacro:if value="${sim_type == 'gazebo'}">
-            <plugin>gazebo_ros2_control/GazeboSystem</plugin>
+            <xacro:if value="${gazebo_version == 'classic'}">
+              <plugin>gazebo_ros2_control/GazeboSystem</plugin>
+            </xacro:if>
+            <xacro:if value="${gazebo_version == 'gazebo'}">
+              <plugin>gz_ros2_control/GazeboSimSystem</plugin>
+            </xacro:if>
           </xacro:if>
         </xacro:if>
         <xacro:unless value="$(arg use_sim_time)">
           <plugin>robot_control/RobotControl</plugin>
+          <param name="error_protection">true</param>
+          <param name="idle_mode_on_stop">true</param>
         </xacro:unless>
       </hardware>

File: pal_sea_arm_description/urdf/arm/arm.ros2_control.xacro (robot description, xacro)
@@ -13,5 +13,5 @@
  -->
 <robot xmlns:xacro="http://ros.org/wiki/xacro">
-  <xacro:macro name="ros2_control_arm" params="name reduction offset_value use_sea_transmission:=false sim_type:=no-simulation">
+  <xacro:macro name="ros2_control_arm" params="name reduction offset_value use_sea_transmission:=false sim_type:=gazebo">
     <joint name="${name}_joint">
       <xacro:if value="${sim_type == 'mujoco-ros2-control'}">
@@ -25,6 +25,11 @@
         <command_interface name="position" />
       </xacro:if>
-      <command_interface name="velocity" />
-      <command_interface name="effort" />
+      <!-- TODO: Remove when moving to Gazebo Harmonic or ROS 2 Jazzy -->
+      <!-- Multiple command interfaces not working on Gazebo Fortress -->
+      <!-- https://github.com/ros-controls/gz_ros2_control/issues/182 -->
+      <xacro:if value="${gazebo_version == 'classic'}">
+        <command_interface name="velocity" />
+        <command_interface name="effort" />
+      </xacro:if>
       <state_interface name="position" />
       <state_interface name="velocity" />
