Commit message: Imported upstream version '2.6.0' of 'upstream'

File: pal_sea_arm_description/urdf/arm/arm.urdf.xacro (robot description, xacro)
@@ -13,6 +13,5 @@
 -->
 <robot xmlns:xacro="http://ros.org/wiki/xacro">
-  <!-- Transmissions file -->
-  <xacro:macro name="pal_sea_arm" params="name parent *origin arm_type tool_changer wrist_model reflect:=1 joint_reflect:=1 arm_1_offset arm_2_offset arm_3_offset arm_4_offset arm_5_offset arm_6_offset arm_7_offset no_safety_eps:=False">
+  <xacro:macro name="pal_sea_arm" params="name parent *origin arm_type tool_changer wrist_model reflect:=1 joint_reflect:=1 arm_1_offset arm_2_offset arm_3_offset arm_4_offset arm_5_offset arm_6_offset arm_7_offset no_safety_eps:=False limits_v2:=False">
     <!-- PROPERTIES -->
     <xacro:property name="arm_eps" value="${0.00 if no_safety_eps else 0.07}"/>
@@ -38,11 +37,4 @@
       <xacro:property name="mesh_folder" value="arm_tiago_sea"/>
     </xacro:if>
-    <!-- Compatibility check with wrist model -->
-    <!-- <xacro:if value="${arm_type == 'tiago-sea' and wrist_model=='spherical-wrist'}">
-      <xacro:error_wrist_not_supported />
-    </xacro:if>
-    <xacro:if value="${arm_type == 'tiago-sea-dual' and wrist_model=='spherical-wrist'}">
-      <xacro:error_wrist_not_supported />
-    </xacro:if> -->
     <!-- INCLUDES -->
     <xacro:include filename="$(find pal_sea_arm_description)/urdf/arm/arm_limits/${arm_type}/arm.limits.xacro"/>
@@ -51,4 +43,5 @@
     <xacro:include filename="$(find pal_sea_arm_description)/urdf/arm/arm_properties/${arm_type}/${wrist_model}.properties.xacro"/>
     <!-- ARM DEFINITION -->
+    <xacro:property name="joint_type" value="${'continuous' if arm_type == 'pal-sea-arm-standalone' else 'revolute'}" />
     <!-- ARM 1 LINK -->
     <link name="${name}_1_link">
@@ -69,12 +62,23 @@
     </link>
     <!-- ARM 1 JOINT -->
-    <joint name="${name}_1_joint" type="revolute">
+    <joint name="${name}_1_joint" type="${joint_type}">
       <xacro:insert_block name="origin"/>
       <parent link="${parent}" />
       <child link="${name}_1_link" />
       <axis xyz="0 0 1" />
-      <limit lower="${arm_1_joint_lb * deg_to_rad}" upper="${arm_1_joint_ub * deg_to_rad}" effort="${arm_1_max_effort}" velocity="${arm_1_max_velocity}" />
+      <xacro:if value="${joint_type == 'continuous'}">
+        <limit effort="${arm_1_max_effort}" velocity="${arm_1_max_velocity}" />
+      </xacro:if>
+      <xacro:if value="${joint_type == 'revolute'}">
+        <xacro:if value="${limits_v2}">
+          <limit lower="${arm_1_joint_lb_v2 * deg_to_rad}" upper="${arm_1_joint_ub_v2 * deg_to_rad}" effort="${arm_1_max_effort}" velocity="${arm_1_max_velocity}" />
+          <safety_controller k_position="${arm_k_position}" k_velocity="${arm_k_velocity}" soft_lower_limit="${arm_1_joint_lb_v2 * deg_to_rad  + arm_eps}" soft_upper_limit="${arm_1_joint_ub_v2 * deg_to_rad  - arm_eps}" />
+        </xacro:if>
+        <xacro:unless value="${limits_v2}">
+          <limit lower="${arm_1_joint_lb * deg_to_rad}" upper="${arm_1_joint_ub * deg_to_rad}" effort="${arm_1_max_effort}" velocity="${arm_1_max_velocity}" />
+          <safety_controller k_position="${arm_k_position}" k_velocity="${arm_k_velocity}" soft_lower_limit="${arm_1_joint_lb * deg_to_rad  + arm_eps}" soft_upper_limit="${arm_1_joint_ub * deg_to_rad  - arm_eps}" />
+        </xacro:unless>
+      </xacro:if>
       <dynamics friction="${arm_friction}" damping="${arm_damping}"/>
-      <safety_controller k_position="${arm_k_position}" k_velocity="${arm_k_velocity}" soft_lower_limit="${arm_1_joint_lb * deg_to_rad  + arm_eps}" soft_upper_limit="${arm_1_joint_ub * deg_to_rad  - arm_eps}" />
     </joint>
     <!-- ARM 2 LINK -->
@@ -123,12 +127,23 @@
     </link>
     <!-- ARM 3 JOINT -->
-    <joint name="${name}_3_joint" type="revolute">
+    <joint name="${name}_3_joint" type="${joint_type}">
       <xacro:origin_joint_3 reflect="${reflect}"/>
       <parent link="${name}_2_link" />
       <child link="${name}_3_link" />
       <axis xyz="0 0 1" />
-      <limit lower="${arm_3_joint_lb * deg_to_rad}" upper="${arm_3_joint_ub * deg_to_rad}" effort="${arm_3_max_effort}" velocity="${arm_3_max_velocity}" />
-      <dynamics friction="${arm_friction}" damping="${arm_damping}"/>
-      <safety_controller k_position="${arm_k_position}" k_velocity="${arm_k_velocity}" soft_lower_limit="${arm_3_joint_lb * deg_to_rad  + arm_eps}" soft_upper_limit="${arm_3_joint_ub * deg_to_rad - arm_eps}" />
+      <xacro:if value="${joint_type == 'continuous'}">
+        <limit effort="${arm_3_max_effort}" velocity="${arm_3_max_velocity}" />
+      </xacro:if>
+      <xacro:if value="${joint_type == 'revolute'}">
+        <xacro:if value="${limits_v2}">
+          <limit lower="${arm_3_joint_lb_v2 * deg_to_rad}" upper="${arm_3_joint_ub_v2 * deg_to_rad}" effort="${arm_3_max_effort}" velocity="${arm_3_max_velocity}" />
+        <safety_controller k_position="${arm_k_position}" k_velocity="${arm_k_velocity}" soft_lower_limit="${arm_3_joint_lb_v2 * deg_to_rad  + arm_eps}" soft_upper_limit="${arm_3_joint_ub_v2 * deg_to_rad - arm_eps}" />
+        </xacro:if>
+        <xacro:unless value="${limits_v2}">
+          <limit lower="${arm_3_joint_lb * deg_to_rad}" upper="${arm_3_joint_ub * deg_to_rad}" effort="${arm_3_max_effort}" velocity="${arm_3_max_velocity}" />
+          <safety_controller k_position="${arm_k_position}" k_velocity="${arm_k_velocity}" soft_lower_limit="${arm_3_joint_lb * deg_to_rad  + arm_eps}" soft_upper_limit="${arm_3_joint_ub * deg_to_rad - arm_eps}" />
+        </xacro:unless>
+      </xacro:if>
+        <dynamics friction="${arm_friction}" damping="${arm_damping}"/>
     </joint>
     <!-- ARM 4 LINK -->
@@ -177,67 +192,80 @@
     </link>
     <!-- ARM 5 JOINT -->
-    <joint name="${name}_5_joint" type="revolute">
+    <joint name="${name}_5_joint" type="${joint_type}">
       <xacro:origin_joint_5 reflect="${reflect}"/>
       <parent link="${name}_4_link" />
       <child link="${name}_5_link" />
       <axis xyz="0 0 1" />
-      <limit lower="${arm_5_joint_lb * deg_to_rad}" upper="${arm_5_joint_ub * deg_to_rad}" effort="${arm_5_max_effort}" velocity="${arm_5_max_velocity}" />
+      <xacro:if value="${joint_type == 'continuous'}">
+        <limit effort="${arm_5_max_effort}" velocity="${arm_5_max_velocity}" />
+      </xacro:if>
+      <xacro:if value="${joint_type == 'revolute'}">
+        <xacro:if value="${limits_v2}">
+          <limit lower="${arm_5_joint_lb_v2 * deg_to_rad}" upper="${arm_5_joint_ub_v2 * deg_to_rad}" effort="${arm_5_max_effort}" velocity="${arm_5_max_velocity}" />
+          <safety_controller k_position="${arm_k_position}" k_velocity="${arm_k_velocity}" soft_lower_limit="${arm_5_joint_lb_v2 * deg_to_rad  + arm_eps}" soft_upper_limit="${arm_5_joint_ub_v2 * deg_to_rad - arm_eps}" />
+        </xacro:if>
+        <xacro:unless value="${limits_v2}">
+          <limit lower="${arm_5_joint_lb * deg_to_rad}" upper="${arm_5_joint_ub * deg_to_rad}" effort="${arm_5_max_effort}" velocity="${arm_5_max_velocity}" />
+          <safety_controller k_position="${arm_k_position}" k_velocity="${arm_k_velocity}" soft_lower_limit="${arm_5_joint_lb * deg_to_rad  + arm_eps}" soft_upper_limit="${arm_5_joint_ub * deg_to_rad - arm_eps}" />
+        </xacro:unless>
+      </xacro:if>
       <dynamics friction="${arm_friction}" damping="${arm_damping}"/>
-      <safety_controller k_position="${arm_k_position}" k_velocity="${arm_k_velocity}" soft_lower_limit="${arm_5_joint_lb * deg_to_rad  + arm_eps}" soft_upper_limit="${arm_5_joint_ub * deg_to_rad - arm_eps}" />
-    </joint>
-    <!-- ARM 6 LINK -->
-    <link name="${name}_6_link">
-      <xacro:inertial_link_6 reflect="${reflect}"/>
-      <visual>
-        <origin xyz="0 0 0" rpy="0 0 0" />
-        <geometry>
-          <mesh filename="package://pal_sea_arm_description/meshes/${mesh_folder}/${wrist_model}/arm_6_link.stl" scale="1 1 ${reflect}" />
-        </geometry>
-        <material name="pal/DarkGrey"/>
-      </visual>
-      <collision>
-        <origin xyz="0 0 0" rpy="0 0 0" />
-        <geometry>
-          <mesh filename="package://pal_sea_arm_description/meshes/${mesh_folder}/${wrist_model}/arm_6_link_collision.stl" scale="1 1 ${reflect}" />
-        </geometry>
-      </collision>
-    </link>
-    <!-- ARM 6 JOINT -->
-    <joint name="${name}_6_joint" type="revolute">
-      <xacro:origin_joint_6 reflect="${reflect}"/>
-      <parent link="${name}_5_link" />
-      <child link="${name}_6_link" />
-      <axis xyz="0 0 ${-1 if wrist_model=='spherical-wrist' else 1}" />
-      <limit lower="${arm_6_joint_lb * deg_to_rad}" upper="${arm_6_joint_ub * deg_to_rad}" effort="${arm_6_max_effort}" velocity="${arm_6_max_velocity}" />
-      <dynamics friction="${arm_friction}" damping="${arm_damping}"/>
-      <safety_controller k_position="${arm_k_position}" k_velocity="${arm_k_velocity}" soft_lower_limit="${arm_6_joint_lb * deg_to_rad  + arm_eps}" soft_upper_limit="${arm_6_joint_ub * deg_to_rad - arm_eps}" />
-    </joint>
-    <!-- ARM 7 LINK -->
-    <link name="${name}_7_link">
-      <xacro:inertial_link_7 reflect="${reflect}"/>
-      <visual>
-        <origin xyz="0 0 0" rpy="0 0 0" />
-        <geometry>
-          <mesh filename="package://pal_sea_arm_description/meshes/${mesh_folder}/${wrist_model}/arm_7_link.stl" scale="1 1 ${reflect}" />
-        </geometry>
-        <material name="pal/DarkGrey"/>
-      </visual>
-      <collision>
-        <origin xyz="0 0 0" rpy="0 0 0" />
-        <geometry>
-          <cylinder radius="0.0375" length="0.0366"/>
-        </geometry>
-      </collision>
-    </link>
-    <!-- ARM 7 JOINT -->
-    <joint name="${name}_7_joint" type="revolute">
-      <xacro:origin_joint_7 reflect="${reflect}"/>
-      <parent link="${name}_6_link" />
-      <child link="${name}_7_link" />
-      <axis xyz="0 0 1" />
-      <limit lower="${arm_7_joint_lb * deg_to_rad}" upper="${arm_7_joint_ub * deg_to_rad}" effort="${arm_7_max_effort}" velocity="${arm_7_max_velocity}" />
-      <dynamics friction="${arm_friction}" damping="${arm_damping}"/>
-      <safety_controller k_position="${arm_k_position}" k_velocity="${arm_k_velocity}" soft_lower_limit="${arm_7_joint_lb * deg_to_rad  + arm_eps}" soft_upper_limit="${arm_7_joint_ub * deg_to_rad - arm_eps}" />
-    </joint>
+    </joint>
+    <xacro:unless value="${wrist_model == 'short-wrist'}">
+      <!-- ARM 6 LINK -->
+      <link name="${name}_6_link">
+        <xacro:inertial_link_6 reflect="${reflect}"/>
+        <visual>
+          <origin xyz="0 0 0" rpy="0 0 0" />
+          <geometry>
+            <mesh filename="package://pal_sea_arm_description/meshes/${mesh_folder}/${wrist_model}/arm_6_link.stl" scale="1 1 ${reflect}" />
+          </geometry>
+          <material name="pal/DarkGrey"/>
+        </visual>
+        <collision>
+          <origin xyz="0 0 0" rpy="0 0 0" />
+          <geometry>
+            <mesh filename="package://pal_sea_arm_description/meshes/${mesh_folder}/${wrist_model}/arm_6_link_collision.stl" scale="1 1 ${reflect}" />
+          </geometry>
+        </collision>
+      </link>
+      <!-- ARM 6 JOINT -->
+      <joint name="${name}_6_joint" type="revolute">
+        <xacro:origin_joint_6 reflect="${reflect}"/>
+        <parent link="${name}_5_link" />
+        <child link="${name}_6_link" />
+        <axis xyz="0 0 ${-1 if wrist_model=='spherical-wrist' else 1}" />
+        <limit lower="${arm_6_joint_lb * deg_to_rad}" upper="${arm_6_joint_ub * deg_to_rad}" effort="${arm_6_max_effort}" velocity="${arm_6_max_velocity}" />
+        <dynamics friction="${arm_friction}" damping="${arm_damping}"/>
+        <safety_controller k_position="${arm_k_position}" k_velocity="${arm_k_velocity}" soft_lower_limit="${arm_6_joint_lb * deg_to_rad  + arm_eps}" soft_upper_limit="${arm_6_joint_ub * deg_to_rad - arm_eps}" />
+      </joint>
+      <!-- ARM 7 LINK -->
+      <link name="${name}_7_link">
+        <xacro:inertial_link_7 reflect="${reflect}"/>
+        <visual>
+          <origin xyz="0 0 0" rpy="0 0 0" />
+          <geometry>
+            <mesh filename="package://pal_sea_arm_description/meshes/${mesh_folder}/${wrist_model}/arm_7_link.stl" scale="1 1 ${reflect}" />
+          </geometry>
+          <material name="pal/DarkGrey"/>
+        </visual>
+        <collision>
+          <origin xyz="0 0 0" rpy="0 0 0" />
+          <geometry>
+            <mesh filename="package://pal_sea_arm_description/meshes/${mesh_folder}/${wrist_model}/arm_7_link_collision.stl" scale="1 1 ${reflect}" />
+          </geometry>
+        </collision>
+      </link>
+      <!-- ARM 7 JOINT -->
+      <joint name="${name}_7_joint" type="revolute">
+        <xacro:origin_joint_7 reflect="${reflect}"/>
+        <parent link="${name}_6_link" />
+        <child link="${name}_7_link" />
+        <axis xyz="0 0 1" />
+        <limit lower="${arm_7_joint_lb * deg_to_rad}" upper="${arm_7_joint_ub * deg_to_rad}" effort="${arm_7_max_effort}" velocity="${arm_7_max_velocity}" />
+        <dynamics friction="${arm_friction}" damping="${arm_damping}"/>
+        <safety_controller k_position="${arm_k_position}" k_velocity="${arm_k_velocity}" soft_lower_limit="${arm_7_joint_lb * deg_to_rad  + arm_eps}" soft_upper_limit="${arm_7_joint_ub * deg_to_rad - arm_eps}" />
+      </joint>
+    </xacro:unless>
     <!--***********************-->
     <!--        TOOL           -->
@@ -247,5 +275,10 @@
       <link name="${name}_tool_link"/>
       <joint name="${name}_tool_joint" type="fixed">
-        <parent link="${name}_7_link" />
+        <xacro:if value="${wrist_model == 'short-wrist'}">
+          <parent link="${name}_5_link" />
+        </xacro:if>
+        <xacro:unless value="${wrist_model == 'short-wrist'}">
+          <parent link="${name}_7_link" />
+        </xacro:unless>
         <child link="${name}_tool_link" />
         <xacro:origin_joint_tool_changer reflect="${reflect}"/>
@@ -254,12 +287,17 @@
     <!-- Without tool changer (tool link just on top of link 7)-->
     <xacro:unless value="${tool_changer}">
-      <link name="${name}_tool_link">
-      </link>
+      <link name="${name}_tool_link"/>
       <joint name="${name}_tool_joint" type="fixed">
-        <parent link="${name}_7_link" />
+        <xacro:if value="${wrist_model == 'short-wrist'}">
+          <parent link="${name}_5_link" />
+        </xacro:if>
+        <xacro:unless value="${wrist_model == 'short-wrist'}">
+          <parent link="${name}_7_link" />
+        </xacro:unless>
         <child link="${name}_tool_link" />
         <origin xyz="0 0 0" rpy="0 ${0 if reflect is 1 else 180 * deg_to_rad} 0.0" />
       </joint>
     </xacro:unless>
+    <!-- GAZEBO PROPERTIES -->
     <gazebo reference="${name}_1_link">
       <material>Gazebo/DarkGrey</material>
@@ -267,4 +305,7 @@
       <mu2>0.9</mu2>
     </gazebo>
+    <gazebo reference="${name}_1_joint">
+      <implicitSpringDamper>1</implicitSpringDamper>
+    </gazebo>
     <gazebo reference="${name}_2_link">
       <material>Gazebo/DarkGrey</material>
@@ -272,4 +313,7 @@
       <mu2>0.9</mu2>
     </gazebo>
+    <gazebo reference="${name}_2_joint">
+      <implicitSpringDamper>1</implicitSpringDamper>
+    </gazebo>
     <gazebo reference="${name}_3_link">
       <material>Gazebo/DarkGrey</material>
@@ -277,4 +321,7 @@
       <mu2>0.9</mu2>
     </gazebo>
+    <gazebo reference="${name}_3_joint">
+      <implicitSpringDamper>1</implicitSpringDamper>
+    </gazebo>
     <gazebo reference="${name}_4_link">
       <material>Gazebo/DarkGrey</material>
@@ -282,4 +329,7 @@
       <mu2>0.9</mu2>
     </gazebo>
+    <gazebo reference="${name}_4_joint">
+      <implicitSpringDamper>1</implicitSpringDamper>
+    </gazebo>
     <gazebo reference="${name}_5_link">
       <material>Gazebo/DarkGrey</material>
@@ -287,4 +337,8 @@
       <mu2>0.9</mu2>
     </gazebo>
+    <gazebo reference="${name}_5_joint">
+      <implicitSpringDamper>1</implicitSpringDamper>
+    </gazebo>
+  <xacro:unless value="${wrist_model == 'short-wrist'}">
     <gazebo reference="${name}_6_link">
       <material>Gazebo/DarkGrey</material>
@@ -292,4 +346,7 @@
       <mu2>0.9</mu2>
     </gazebo>
+    <gazebo reference="${name}_6_joint">
+      <implicitSpringDamper>1</implicitSpringDamper>
+    </gazebo>
     <gazebo reference="${name}_7_link">
       <material>Gazebo/DarkGrey</material>
@@ -297,30 +354,13 @@
       <mu2>0.9</mu2>
     </gazebo>
+    <gazebo reference="${name}_7_joint">
+      <implicitSpringDamper>1</implicitSpringDamper>
+      <provideFeedback>1</provideFeedback>
+    </gazebo>
+  </xacro:unless>
     <gazebo reference="${name}_tool_link">
       <material>Gazebo/DarkGrey</material>
       <mu1>0.9</mu1>
       <mu2>0.9</mu2>
-    </gazebo>
-    <gazebo reference="${name}_1_joint">
-      <implicitSpringDamper>1</implicitSpringDamper>
-    </gazebo>
-    <gazebo reference="${name}_2_joint">
-      <implicitSpringDamper>1</implicitSpringDamper>
-    </gazebo>
-    <gazebo reference="${name}_3_joint">
-      <implicitSpringDamper>1</implicitSpringDamper>
-    </gazebo>
-    <gazebo reference="${name}_4_joint">
-      <implicitSpringDamper>1</implicitSpringDamper>
-    </gazebo>
-    <gazebo reference="${name}_5_joint">
-      <implicitSpringDamper>1</implicitSpringDamper>
-    </gazebo>
-    <gazebo reference="${name}_6_joint">
-      <implicitSpringDamper>1</implicitSpringDamper>
-    </gazebo>
-    <gazebo reference="${name}_7_joint">
-      <implicitSpringDamper>1</implicitSpringDamper>
-      <provideFeedback>1</provideFeedback>
     </gazebo>
   </xacro:macro>

File: pal_sea_arm_description/urdf/arm/arm_limits/pal-sea-arm-standalone/arm.limits.xacro (robot description, xacro)
@@ -6,10 +6,6 @@
   <xacro:property name="arm_k_velocity" value="20"/>
   <!-- Joint limits -->
-  <xacro:property name="arm_1_joint_ub" value="148.97" />
-  <xacro:property name="arm_1_joint_lb" value="-148.97" />
   <xacro:property name="arm_2_joint_ub" value="63.03" />
   <xacro:property name="arm_2_joint_lb" value="-139.8" />
-  <xacro:property name="arm_3_joint_ub" value="148.97" />
-  <xacro:property name="arm_3_joint_lb" value="-148.97" />
   <xacro:property name="arm_4_joint_ub" value="63.03" />
   <xacro:property name="arm_4_joint_lb" value="-139.8" />

File: pal_sea_arm_description/urdf/arm/arm_limits/pal-sea-arm-standalone/spherical-wrist.limits.xacro (robot description, xacro)
@@ -1,10 +1,8 @@
 <robot xmlns:xacro="http://ros.org/wiki/xacro">
   <!-- Joint limits -->
-  <xacro:property name="arm_5_joint_ub" value="210" />
-  <xacro:property name="arm_5_joint_lb" value="-90" />
-  <xacro:property name="arm_6_joint_ub" value="114.59" />
-  <xacro:property name="arm_6_joint_lb" value="-114.59" />
-  <xacro:property name="arm_7_joint_ub" value="148.97" />
-  <xacro:property name="arm_7_joint_lb" value="-148.97" />
+  <xacro:property name="arm_6_joint_ub" value="172" />
+  <xacro:property name="arm_6_joint_lb" value="-98" />
+  <xacro:property name="arm_7_joint_ub" value="140" />
+  <xacro:property name="arm_7_joint_lb" value="-140" />
   <!-- Velocity limits -->
   <xacro:property name="arm_5_max_velocity" value="3.95" />

File: pal_sea_arm_description/urdf/arm/arm_limits/pal-sea-arm-standalone/straight-wrist.limits.xacro (robot description, xacro)
@@ -1,10 +1,8 @@
 <robot xmlns:xacro="http://ros.org/wiki/xacro">
   <!-- Joint limits -->
-  <xacro:property name="arm_5_joint_ub" value="148.97" />
-  <xacro:property name="arm_5_joint_lb" value="-148.97" />
   <xacro:property name="arm_6_joint_ub" value="114.59" />
   <xacro:property name="arm_6_joint_lb" value="-114.59" />
-  <xacro:property name="arm_7_joint_ub" value="148.97" />
-  <xacro:property name="arm_7_joint_lb" value="-148.97" />
+  <xacro:property name="arm_7_joint_ub" value="140" />
+  <xacro:property name="arm_7_joint_lb" value="-140" />
   <!-- Velocity limits -->
   <xacro:property name="arm_5_max_velocity" value="3.95" />

File: pal_sea_arm_description/urdf/arm/arm_limits/tiago-pro/spherical-wrist.limits.xacro (robot description, xacro)
@@ -5,6 +5,9 @@
   <xacro:property name="arm_6_joint_ub" value="172" />
   <xacro:property name="arm_6_joint_lb" value="-108" />
-  <xacro:property name="arm_7_joint_ub" value="150" />
-  <xacro:property name="arm_7_joint_lb" value="-150" />
+  <xacro:property name="arm_7_joint_ub" value="140" />
+  <xacro:property name="arm_7_joint_lb" value="-140" />
+  <!-- Joint limtis v2 -->
+  <xacro:property name="arm_5_joint_ub_v2" value="${220 if joint_reflect == 1 else 100}" />
+  <xacro:property name="arm_5_joint_lb_v2" value="${-100 if joint_reflect == 1 else -220}" />
   <!-- Velocity limits -->
   <xacro:property name="arm_5_max_velocity" value="3.95" />
